File: LeonardoBB.kicad_pcb (KiCad board)
At the start: 2 copper layers, 48 x 58 mm, 43 parts, among them J1 USB_B_Micro, J2 Conn_01x17, J3 Conn_01x17, J4 I2C, Q1 Q_PMOS_GSD, Q2 Q_DUAL_PMOS_S1G1D2S2G2D1, SW1 SW_SPDT, U1 ATmega32U4-MU, U2 LMV358, U3 NCP1117-5.0_SOT223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

Commit message: Add reset switch
Parts:
- added SW2: SW_Push, Button_Switch_SMD:SW_SPST_PTS810, B.Cu at (130.5, 124.7)
- moved D2 1.05 mm to (135.7, 125.6)
Routing:
- net RESET: track 28.8 -> 51.8 mm, vias 1 -> 2
- net GND: track 296.8 -> 303.4 mm
- net +5V: track 135.5 -> 130.7 mm, vias 4 -> 5
- net Net-(D2-Pad2): track 10.7 -> 9.91 mm
Other:
- board text added: "D13"
- board text added: "Reset"
